Commit message: both base and arm can be controlled at the same time

File: install/share/ombot_description/urdf/arm/ombot_arm.ros2_control.xacro (robot description, xacro)
@@ -4,5 +4,5 @@
     <ros2_control name="${name}" type="system">
       <hardware>
-        <plugin>ros2_control_demo_example_7/OMBotHardware</plugin>
+        <plugin>ombot_hardware/OMBotArmSystem</plugin>
         <param name="port">/dev/ttyUSB0</param>
         <param name="baudrate">1000000</param>

File: install/share/ombot_description/urdf/arm/ombot_arm_description.urdf.xacro (robot description, xacro)
@@ -9,12 +9,12 @@
         <!-- <mesh filename="package://ros2_control_demos/meshes/link_1.stl" scale="0.001 0.001 0.001"/>
         <mesh filename="package://ombot_description/meshes/link6.stl"/> -->
-        <mesh filename="/home/frank/frank_ws/src/ombot_description/meshes/arm/link1.stl" scale="0.001 0.001 0.001"/>
-      </geometry>
-      <material name="grey"/>
-    </visual>
-    <collision>
-      <origin xyz="0 0 0" rpy="0 0 0"/>
-      <geometry>
-        <mesh filename="/home/frank/frank_ws/src/ombot_description/meshes/arm/link1.stl" scale="0.001 0.001 0.001"/>
+        <mesh filename="package://ombot_description/meshes/arm/link1.stl" scale="0.001 0.001 0.001"/>
+      </geometry>
+      <material name="grey"/>
+    </visual>
+    <collision>
+      <origin xyz="0 0 0" rpy="0 0 0"/>
+      <geometry>
+        <mesh filename="package://ombot_description/meshes/arm/link1.stl" scale="0.001 0.001 0.001"/>
       </geometry>
     </collision>
@@ -40,12 +40,12 @@
       <origin xyz="0 0 0" rpy="0 0 0"/>
       <geometry>
-        <mesh filename="/home/frank/frank_ws/src/ombot_description/meshes/arm/link2.stl" scale="0.001 0.001 0.001"/>
-      </geometry>
-      <material name="grey"/>
-    </visual>
-    <collision>
-      <origin xyz="0 0 0" rpy="0 0 0"/>
-      <geometry>
-        <mesh filename="/home/frank/frank_ws/src/ombot_description/meshes/arm/link2.stl" scale="0.001 0.001 0.001"/>
+        <mesh filename="package://ombot_description/meshes/arm/link2.stl" scale="0.001 0.001 0.001"/>
+      </geometry>
+      <material name="grey"/>
+    </visual>
+    <collision>
+      <origin xyz="0 0 0" rpy="0 0 0"/>
+      <geometry>
+        <mesh filename="package://ombot_description/meshes/arm/link2.stl" scale="0.001 0.001 0.001"/>
       </geometry>
     </collision>
@@ -72,12 +72,12 @@
       <origin xyz="0 0 0" rpy="0 0 0"/>
       <geometry>
-        <mesh filename="/home/frank/frank_ws/src/ombot_description/meshes/arm/link3.stl" scale="0.001 0.001 0.001"/>
-      </geometry>
-      <material name="grey"/>
-    </visual>
-    <collision>
-      <origin xyz="0 0 0" rpy="0 0 0"/>
-      <geometry>
-        <mesh filename="/home/frank/frank_ws/src/ombot_description/meshes/arm/link3.stl" scale="0.001 0.001 0.001"/>
+        <mesh filename="package://ombot_description/meshes/arm/link3.stl" scale="0.001 0.001 0.001"/>
+      </geometry>
+      <material name="grey"/>
+    </visual>
+    <collision>
+      <origin xyz="0 0 0" rpy="0 0 0"/>
+      <geometry>
+        <mesh filename="package://ombot_description/meshes/arm/link3.stl" scale="0.001 0.001 0.001"/>
       </geometry>
     </collision>
@@ -104,12 +104,12 @@
       <origin xyz="0 0 0" rpy="0 0 0"/>
       <geometry>
-        <mesh filename="/home/frank/frank_ws/src/ombot_description/meshes/arm/link4.stl" scale="0.001 0.001 0.001"/>
-      </geometry>
-      <material name="grey"/>
-    </visual>
-    <collision>
-      <origin xyz="0 0 0" rpy="0 0 0"/>
-      <geometry>
-        <mesh filename="/home/frank/frank_ws/src/ombot_description/meshes/arm/link4.stl" scale="0.001 0.001 0.001"/>
+        <mesh filename="package://ombot_description/meshes/arm/link4.stl" scale="0.001 0.001 0.001"/>
+      </geometry>
+      <material name="grey"/>
+    </visual>
+    <collision>
+      <origin xyz="0 0 0" rpy="0 0 0"/>
+      <geometry>
+        <mesh filename="package://ombot_description/meshes/arm/link4.stl" scale="0.001 0.001 0.001"/>
       </geometry>
     </collision>
@@ -136,12 +136,12 @@
       <origin xyz="0 0 0" rpy="0 0 0"/>
       <geometry>
-        <mesh filename="/home/frank/frank_ws/src/ombot_description/meshes/arm/link5.stl" scale="0.001 0.001 0.001"/>
-      </geometry>
-      <material name="grey"/>
-    </visual>
-    <collision>
-      <origin xyz="0 0 0" rpy="0 0 0"/>
-      <geometry>
-        <mesh filename="/home/frank/frank_ws/src/ombot_description/meshes/arm/link5.stl" scale="0.001 0.001 0.001"/>
+        <mesh filename="package://ombot_description/meshes/arm/link5.stl" scale="0.001 0.001 0.001"/>
+      </geometry>
+      <material name="grey"/>
+    </visual>
+    <collision>
+      <origin xyz="0 0 0" rpy="0 0 0"/>
+      <geometry>
+        <mesh filename="package://ombot_description/meshes/arm/link5.stl" scale="0.001 0.001 0.001"/>
       </geometry>
     </collision>
@@ -168,12 +168,12 @@
       <origin xyz="0 0 0" rpy="0 0 0"/>
       <geometry>
-        <mesh filename="/home/frank/frank_ws/src/ombot_description/meshes/arm/link6.stl" scale="0.001 0.001 0.001"/>
-      </geometry>
-      <material name="grey"/>
-    </visual>
-    <collision>
-      <origin xyz="0 0 0" rpy="0 0 0"/>
-      <geometry>
-        <mesh filename="/home/frank/frank_ws/src/ombot_description/meshes/arm/link6.stl" scale="0.001 0.001 0.001"/>
+        <mesh filename="package://ombot_description/meshes/arm/link6.stl" scale="0.001 0.001 0.001"/>
+      </geometry>
+      <material name="grey"/>
+    </visual>
+    <collision>
+      <origin xyz="0 0 0" rpy="0 0 0"/>
+      <geometry>
+        <mesh filename="package://ombot_description/meshes/arm/link6.stl" scale="0.001 0.001 0.001"/>
       </geometry>
     </collision>
@@ -200,5 +200,5 @@
       <origin xyz="0.0 0.0 0.0" rpy="0 0 0" />
       <geometry>
-        <mesh filename="/home/frank/frank_ws/src/ombot_description/meshes/arm/end_link.stl" scale="0.001 0.001 0.001"/>
+        <mesh filename="package://ombot_description/meshes/arm/end_link.stl" scale="0.001 0.001 0.001"/>
       </geometry>
       <material name="grey"/>
@@ -207,5 +207,5 @@
       <origin xyz="0.0 0.0 0.0" rpy="0 0 0" />
       <geometry>
-        <mesh filename="/home/frank/frank_ws/src/ombot_description/meshes/arm/end_link.stl" scale="0.001 0.001 0.001"/>
+        <mesh filename="package://ombot_description/meshes/arm/end_link.stl" scale="0.001 0.001 0.001"/>
       </geometry>
     </collision>

File: install/share/ombot_description/urdf/arm/ombot_arm_module.urdf.xacro (robot description, xacro)
@@ -5,5 +5,5 @@
   <xacro:include filename="/home/frank/frank_ws/src/ombot_description/urdf/arm/ombot_arm_description.urdf.xacro"/>
   <xacro:include filename="/home/frank/frank_ws/src/ombot_description/urdf/arm/ombot_arm.transmission.xacro"/>
-  <xacro:include filename="/home/frank/frank_ws/src/ombot_description/urdf/arm/ombot_arm.ros2_control.xacro"/>
+  <!-- <xacro:include filename="/home/frank/frank_ws/src/ombot_description/urdf/arm/ombot_arm.ros2_control.xacro"/> -->
   <!--
     Macro to place/mount the arm on any parent link.

File: install/share/ombot_description/urdf/base/mecanum_base.urdf.xacro (robot description, xacro)
@@ -6,5 +6,5 @@
       <xacro:arg name="robot_name" default="robot_3d"/>
       <xacro:arg name="prefix" default=""/>
-      <xacro:arg name="use_gazebo" default="false"/>
+      <!-- <xacro:arg name="use_gazebo" default="false"/> -->
       <!-- <xacro:include filename="$(dirname ${xacro_dir})/mech/robot_3d_base.urdf.xacro"/> -->
       <!-- <xacro:include filename="package://ombot_description/urdf/base/mech/robot_3d_base.urdf.xacro"/> -->
@@ -15,7 +15,7 @@
       <xacro:include filename="/home/frank/frank_ws/src/ombot_description/urdf/base/sensors/imu.urdf.xacro"/>
       <!-- <xacro:include filename="$(find-pkg-share ombot_description)/urdf/base/mech/robot_3d_base.urdf.xacro"/> -->
-      <!-- <xacro:include filename="$(find ombot_description)/urdf/base/mech/robot_3d_base.urdf.xacro"/> -->
-      <!-- <xacro:include filename="$(find ombot_description)/urdf/base/mech/mecanum_wheel.urdf.xacro"/> -->
-      <!-- <xacro:include filename="$(find ombot_description)/urdf/base/sensors/rgbd_camera.urdf.xacro"/>
+      <!-- <xacro:include filename="$(find ombot_description)/urdf/base/mech/robot_3d_base.urdf.xacro"/>
+      <xacro:include filename="$(find ombot_description)/urdf/base/mech/mecanum_wheel.urdf.xacro"/>
+      <xacro:include filename="$(find ombot_description)/urdf/base/sensors/rgbd_camera.urdf.xacro"/>
       <xacro:include filename="$(find ombot_description)/urdf/base/sensors/lidar.urdf.xacro"/>
       <xacro:include filename="$(find ombot_description)/urdf/base/sensors/imu.urdf.xacro"/> -->
@@ -34,10 +34,10 @@
       <xacro:mecanum_wheel
         prefix="$(arg prefix)"
-        side="back_left"
+        side="rear_left"
         x_reflect="-1"
         y_reflect="1"/>
       <xacro:mecanum_wheel
         prefix="$(arg prefix)"
-        side="back_right"
+        side="rear_right"
         x_reflect="-1"
         y_reflect="-1"/>

File: install/share/ombot_description/urdf/base/mech/mecanum_wheel.urdf.xacro (robot description, xacro)
@@ -12,5 +12,5 @@
         <origin xyz="0 0 0" rpy="${pi/2} 0 0"/>
         <geometry>
-          <mesh filename="/home/frank/frank_ws/src/ombot_description/meshes/base/${side}_wheel_X3.STL" scale="2.15 2.15 2.15"/>
+          <mesh filename="package://ombot_description/meshes/base/${side}_wheel_X3.STL" scale="2.15 2.15 2.15"/>
         </geometry>
         <material name="dark_gray">

File: install/share/ombot_description/urdf/base/mech/robot_3d_base.urdf.xacro (robot description, xacro)
@@ -20,5 +20,7 @@
     <visual>
         <geometry>
-            <mesh filename="/home/frank/frank_ws/src/ombot_description/meshes/base/base_link_X3.STL"
+            <!-- <mesh filename="/home/frank/frank_ws/src/ombot_description/meshes/base/base_link_X3.STL"
+                  scale="${mesh_sx} ${mesh_sy} ${mesh_sz}"/> -->
+            <mesh filename="package://ombot_description/meshes/base/base_link_X3.STL"
                   scale="${mesh_sx} ${mesh_sy} ${mesh_sz}"/>
         </geometry>

File: install/share/ombot_description/urdf/base/sensors/lidar.urdf.xacro (robot description, xacro)
@@ -6,5 +6,5 @@
     parent:='base_link'
     frame_id:='laser_frame'
-    mesh_file:='/home/frank/frank_ws/src/ombot_description/meshes/base/rplidar_s2.stl'
+    mesh_file:='package://ombot_description/meshes/base/rplidar_s2.stl'
     xyz_offset:='0 0 0.0825'
     rpy_offset:='0 0 0'

File: install/share/ombot_description/urdf/base/sensors/rgbd_camera.urdf.xacro (robot description, xacro)
@@ -6,5 +6,5 @@
     camera_name:='cam_1'
     parent:='base_link'
-    mesh_file:='/home/frank/frank_ws/src/ombot_description/meshes/base/d435.stl'
+    mesh_file:='package://ombot_description/meshes/base/d435.stl'
     xyz_offset:='0.105 0 0.05'
     rpy_offset:='0 -0.50 0'

File: install/share/ombot_description/urdf/ombot.urdf.xacro (robot description, xacro)
@@ -38,5 +38,5 @@
     </hardware>
     <!-- ARM HARDWARE -->
-    <hardware>
+    <!-- <hardware>
       <plugin>ombot_hardware/OMBotArmSystem</plugin>
       <param name="port">/dev/ttyUSB0</param>
@@ -44,44 +44,23 @@
       <param name="default_mode">effort</param>
       <param name="simulate">false</param>
-      <!-- Arm hardware params here if needed -->
-    </hardware>
+    </hardware> -->
     <!-- Exported joints/interfaces.
          Keep these in sync with your geometry macros’ joint names. -->
-    <!-- <joint name="front_left_wheel_joint">
-      <command_interface name="velocity"/>
-      <state_interface   name="velocity"/>
-      <state_interface   name="position"/>
-    </joint>
-    <joint name="front_right_wheel_joint">
-      <command_interface name="velocity"/>
-      <state_interface   name="velocity"/>
-      <state_interface   name="position"/>
-    </joint>
-    <joint name="back_left_wheel_joint">
-      <command_interface name="velocity"/>
-      <state_interface   name="velocity"/>
-      <state_interface   name="position"/>
-    </joint>
-    <joint name="back_right_wheel_joint">
-      <command_interface name="velocity"/>
-      <state_interface   name="velocity"/>
-      <state_interface   name="position"/>
-    </joint> -->
-    <joint name="fl_wheel_joint">
+    <joint name="front_left_wheel_joint">
       <command_interface name="velocity"/>
       <state_interface name="position"/>
       <state_interface name="velocity"/>
     </joint>
-    <joint name="fr_wheel_joint">
+    <joint name="front_right_wheel_joint">
       <command_interface name="velocity"/>
       <state_interface name="position"/>
       <state_interface name="velocity"/>
     </joint>
-    <joint name="rl_wheel_joint">
+    <joint name="rear_left_wheel_joint">
       <command_interface name="velocity"/>
       <state_interface name="position"/>
       <state_interface name="velocity"/>
     </joint>
-    <joint name="rr_wheel_joint">
+    <joint name="rear_right_wheel_joint">
       <command_interface name="velocity"/>
       <state_interface name="position"/>
@@ -89,5 +68,5 @@
     </joint>
     <!-- Arm joints (prefix “arm_” because of the module call above) -->
-    <joint name="arm_joint_1">
+    <!-- <joint name="arm_joint_1">
       <command_interface name="position"/>
       <command_interface name="effort"/>
@@ -130,5 +109,5 @@
       <state_interface   name="velocity"/>
       <state_interface   name="effort"/>
-    </joint>
+    </joint> -->
   </ros2_control>
 </robot>

File: src/ombot_description/urdf/ombot.urdf.xacro (robot description, xacro)
@@ -38,5 +38,5 @@
     </hardware>
     <!-- ARM HARDWARE -->
-    <hardware>
+    <!-- <hardware>
       <plugin>ombot_hardware/OMBotArmSystem</plugin>
       <param name="port">/dev/ttyUSB0</param>
@@ -44,24 +44,23 @@
       <param name="default_mode">effort</param>
       <param name="simulate">false</param>
-      <!-- Arm hardware params here if needed -->
-    </hardware>
+    </hardware> -->
     <!-- Exported joints/interfaces.
          Keep these in sync with your geometry macros’ joint names. -->
-    <joint name="fl_wheel_joint">
+    <joint name="front_left_wheel_joint">
       <command_interface name="velocity"/>
       <state_interface name="position"/>
       <state_interface name="velocity"/>
     </joint>
-    <joint name="fr_wheel_joint">
+    <joint name="front_right_wheel_joint">
       <command_interface name="velocity"/>
       <state_interface name="position"/>
       <state_interface name="velocity"/>
     </joint>
-    <joint name="rl_wheel_joint">
+    <joint name="rear_left_wheel_joint">
       <command_interface name="velocity"/>
       <state_interface name="position"/>
       <state_interface name="velocity"/>
     </joint>
-    <joint name="rr_wheel_joint">
+    <joint name="rear_right_wheel_joint">
       <command_interface name="velocity"/>
       <state_interface name="position"/>
@@ -69,5 +68,5 @@
     </joint>
     <!-- Arm joints (prefix “arm_” because of the module call above) -->
-    <joint name="arm_joint_1">
+    <!-- <joint name="arm_joint_1">
       <command_interface name="position"/>
       <command_interface name="effort"/>
@@ -110,5 +109,5 @@
       <state_interface   name="velocity"/>
       <state_interface   name="effort"/>
-    </joint>
+    </joint> -->
   </ros2_control>
 </robot>
