Commit message: finished the resolved rate controller

File: src/ombot_description/urdf/arm/ombot_arm_description.urdf.xacro (robot description, xacro)
@@ -186,4 +186,28 @@
     </inertial>
   </link>
+  <!-- Camera body frame mounted to link_6 -->
+  <link name="camera_link">
+    <visual>
+      <origin xyz="0 0 0" rpy="0 0 0"/>
+      <geometry>
+        <box size="0.055 0.135 0.03"/>
+      </geometry>
+      <material name="black"/>
+    </visual>
+  </link>
+  <joint name="camera_mount_joint" type="fixed">
+    <parent link="link_6"/>
+    <!-- Adjust these to your actual bracket offsets on link_6 -->
+    <child link="camera_link"/>
+    <origin xyz="0.08 -0.045 -0.035" rpy="0 0 0"/>
+  </joint>
+  <!-- Standard ROS optical frame: z forward, x right, y down (REP 103) -->
+  <link name="camera_optical_frame"/>
+  <joint name="camera_optical_joint" type="fixed">
+    <parent link="camera_link"/>
+    <child link="camera_optical_frame"/>
+    <!-- This rotation converts a conventional 'camera_link' to an optical frame -->
+    <origin xyz="0 0 0" rpy="-1.57079632679 0 -1.57079632679"/>
+  </joint>
   <!-- Joint 6 -->
   <joint name="joint_6" type="revolute">

Commit message: gripper works on the python script

File: src/ombot_description/urdf/arm/ombot_arm_description.urdf.xacro (robot description, xacro)
@@ -22,6 +22,6 @@
       <origin xyz="0.00023 0.00000 0.06223" rpy="0 0 0"/>
       <mass value="0.85644"/>
-      <inertia ixx="1.0" ixy="0.0" ixz="0.0" iyy="1.0" iyz="0.0" izz="1.0" />
-      <!--<inertia ixx="0.00121064" ixy="0.0" ixz="0.00001100" iyy="0.00120886" iyz="0.0" izz="0.00038103" />-->
+      <!-- <inertia ixx="1.0" ixy="0.0" ixz="0.0" iyy="1.0" iyz="0.0" izz="1.0" /> -->
+      <inertia ixx="0.00121064" ixy="0.0" ixz="0.00001100" iyy="0.00120886" iyz="0.0" izz="0.00038103" />
     </inertial>
   </link>
@@ -54,6 +54,6 @@
       <!--<origin xyz="0.00000 -0.06820 -0.00117" rpy="0 0 0"/>-->
       <mass value="0.94658"/>
-      <inertia ixx="1.0" ixy="0.0" ixz="0.0" iyy="1.0" iyz="0.0" izz="1.0" />
-      <!--<inertia ixx="0.00152547" ixy="0.0" ixz="0.0" iyy="0.00045954" iyz="-0.00001086" izz="0.00151740" />-->
+      <!-- <inertia ixx="1.0" ixy="0.0" ixz="0.0" iyy="1.0" iyz="0.0" izz="1.0" /> -->
+      <inertia ixx="0.00152547" ixy="0.0" ixz="0.0" iyy="0.00045954" iyz="-0.00001086" izz="0.00151740" />
     </inertial>
   </link>
@@ -86,6 +86,6 @@
       <!--<origin xyz="-0.01232 -0.05731 -0.05876" rpy="0 0 0"/>-->
       <mass value="1.30260"/>
-      <inertia ixx="1.0" ixy="0.0" ixz="0.0" iyy="1.0" iyz="0.0" izz="1.0" />
-      <!--<inertia ixx="0.01111021" ixy="0.00001331" ixz="-0.00134208" iyy="0.01046642" iyz="0.00016235" izz="0.00202081" />-->
+      <!-- <inertia ixx="1.0" ixy="0.0" ixz="0.0" iyy="1.0" iyz="0.0" izz="1.0" /> -->
+      <inertia ixx="0.01111021" ixy="0.00001331" ixz="-0.00134208" iyy="0.01046642" iyz="0.00016235" izz="0.00202081" />
     </inertial>
   </link>
@@ -118,6 +118,6 @@
       <!--<origin xyz="-0.07025 0.00034 -0.00021" rpy="0 0 0"/>-->
       <mass value="1.15977"/>
-      <inertia ixx="1.0" ixy="0.0" ixz="0.0" iyy="1.0" iyz="0.0" izz="1.0" />
-      <!--<inertia ixx="0.00096726" ixy="0.00004383" ixz="-0.00002771" iyy="0.00318801" iyz="0.00000627" izz="0.00341484" />-->
+      <!-- <inertia ixx="1.0" ixy="0.0" ixz="0.0" iyy="1.0" iyz="0.0" izz="1.0" /> -->
+      <inertia ixx="0.00096726" ixy="0.00004383" ixz="-0.00002771" iyy="0.00318801" iyz="0.00000627" izz="0.00341484" />
     </inertial>
   </link>
@@ -150,6 +150,6 @@
       <!--<origin xyz="-0.00658 -0.04717 0.00002" rpy="0 0 0"/>-->
       <mass value="0.44688"/>
-      <inertia ixx="1.0" ixy="0.0" ixz="0.0" iyy="1.0" iyz="0.0" izz="1.0" />
-      <!--<inertia ixx="0.00030285" ixy="0.00000761" ixz="0.00000031" iyy="0.00022339" iyz="-0.00000001" izz="0.00039766" />-->
+      <!-- <inertia ixx="1.0" ixy="0.0" ixz="0.0" iyy="1.0" iyz="0.0" izz="1.0" /> -->
+      <inertia ixx="0.00030285" ixy="0.00000761" ixz="0.00000031" iyy="0.00022339" iyz="-0.00000001" izz="0.00039766" />
     </inertial>
   </link>
@@ -182,6 +182,6 @@
       <!--<origin xyz="-0.05469 0.00043 0.00000" rpy="0 0 0"/>-->
       <mass value="0.43273"/>
-      <inertia ixx="1.0" ixy="0.0" ixz="0.0" iyy="1.0" iyz="0.0" izz="1.0" />
-      <!--<inertia ixx="0.00021512" ixy="0.00001009" ixz="0.00000000" iyy="0.00042827" iyz="0.00000000" izz="0.00051436" />-->
+      <!-- <inertia ixx="1.0" ixy="0.0" ixz="0.0" iyy="1.0" iyz="0.0" izz="1.0" /> -->
+      <inertia ixx="0.00021512" ixy="0.00001009" ixz="0.00000000" iyy="0.00042827" iyz="0.00000000" izz="0.00051436" />
     </inertial>
   </link>
@@ -237,6 +237,6 @@
       <origin xyz="0.00337 0.00000 0.00000" rpy="0 0 0"/>
       <mass value="0.01919"/>
-      <inertia ixx="1.0" ixy="0.0" ixz="0.0" iyy="1.0" iyz="0.0" izz="1.0" />
-      <!--<inertia ixx="0.00000938" ixy="0.0" ixz="0.0" iyy="0.00000338" iyz="0.0" izz="0.00000635" />-->
+      <!-- <inertia ixx="1.0" ixy="0.0" ixz="0.0" iyy="1.0" iyz="0.0" izz="1.0" /> -->
+      <inertia ixx="0.00000938" ixy="0.0" ixz="0.0" iyy="0.00000338" iyz="0.0" izz="0.00000635" />
     </inertial>
   </link>

File: src/ombot_description/urdf/base/mech/mecanum_wheel.urdf.xacro (robot description, xacro)
@@ -1,10 +1,10 @@
 <?xml version="1.0"?>
 <robot xmlns:xacro="http://www.ros.org/wiki/xacro">
-  <xacro:property name="wheel_radius" value="0.06985" />
+  <xacro:property name="wheel_radius" value="0.05985" />
   <xacro:property name="wheel_separation" value="0.51" />
   <xacro:property name="wheel_width" value="0.0508" />
   <xacro:property name="wheel_mass" value="9.1" />
-  <xacro:property name="wheel_xoff" value="0.197" />
-  <xacro:property name="wheel_yoff" value="-0.01" />
+  <xacro:property name="wheel_xoff" value="0.2" />
+  <xacro:property name="wheel_yoff" value="0.008" />
   <xacro:macro name="mecanum_wheel" params="prefix side x_reflect y_reflect">
     <link name="${prefix}${side}_wheel_link">

File: src/ombot_description/urdf/base/mech/robot_3d_base.urdf.xacro (robot description, xacro)
@@ -12,15 +12,16 @@
 <xacro:property name="base_size_z" value="${total_height - 2*wheel_radius}"/> <!-- = 0.21 - 2*0.057 = 0.096 -->
 <!-- No offset needed when base_link is centered -->
-<xacro:property name="base_x_offset" value="-0.0095"/>
-<xacro:property name="base_z_offset" value="0.0096"/>
+<xacro:property name="base_x_offset" value="-0.018"/>
+<xacro:property name="base_z_offset" value="0.001"/>
+<xacro:property name="base_y_offset" value="-0.013"/>
 <xacro:property name="base_mass" value="4.6" />
-<xacro:macro name="robot_3d_base" params="prefix mesh_sx:=2.44 mesh_sy:=3.44 mesh_sz:=1.9871">
+<xacro:macro name="robot_3d_base" params="prefix mesh_sx:=0.001 mesh_sy:=0.001 mesh_sz:=0.001">
   <link name="${prefix}base_footprint"/>
   <link name="${prefix}base_link">
     <visual>
         <geometry>
-            <!-- <mesh filename="/home/frank/frank_ws/src/ombot_description/meshes/base/base_link_X3.STL"
+            <!-- <mesh filename="/home/frank/frank_ws/src/ombot_description/meshes/base/frank_base.stl"
                   scale="${mesh_sx} ${mesh_sy} ${mesh_sz}"/> -->
-            <mesh filename="package://ombot_description/meshes/base/base_link_X3.STL"
+            <mesh filename="package://ombot_description/meshes/base/frank_base.STL"
                   scale="${mesh_sx} ${mesh_sy} ${mesh_sz}"/>
         </geometry>
@@ -28,5 +29,5 @@
           <color rgba="1 1 1 1"/>
         </material>
-        <origin xyz="${base_x_offset} 0 ${base_z_offset}" rpy="0 0 0"/>
+        <origin xyz="${base_x_offset} ${base_y_offset} ${base_z_offset}" rpy="1.5708 0 0"/>
     </visual>
     <collision>
@@ -34,8 +35,8 @@
             <box size="${base_size_x} ${base_size_y} ${base_size_z}"/>
         </geometry>
-        <origin xyz="${base_x_offset} 0 ${base_size_z/2 + wheel_radius/4}" rpy="0 0 0"/>
+        <origin xyz="${base_x_offset} ${base_y_offset} ${base_size_z/2 + wheel_radius/4}" rpy="0 0 0"/>
     </collision>
     <inertial>
-        <origin xyz="${base_x_offset} 0 ${base_size_z/2 + wheel_radius/4}" rpy="0 0 0"/>
+        <origin xyz="${base_x_offset} ${base_y_offset} ${base_size_z/2 + wheel_radius/4}" rpy="0 0 0"/>
         <mass value="${base_mass}"/>
         <inertia

File: src/ombot_description/urdf/ombot.urdf.xacro (robot description, xacro)
@@ -7,5 +7,5 @@
     prefix=""
     sep_x="0.40"
-    sep_y="0.30"
+    sep_y="0.70"
     wheel_radius="0.05"/>
   <!-- Arm geometry (MACRO LIB) -->
@@ -14,5 +14,5 @@
   <xacro:ombot_arm_module
     parent="base_link"
-    mount_xyz="0 0 0.01"
+    mount_xyz="0.145 0.0 0.1"
     mount_rpy="0 0 0"
     prefix=""/>
@@ -64,5 +64,5 @@
     <hardware>
       <plugin>ombot_hardware/OMBotArmSystem</plugin>
-      <param name="port">/dev/ttyUSB0</param>
+      <param name="port">/dev/arm_u2d2</param>
       <param name="baudrate">1000000</param>
       <param name="default_mode">effort</param>
@@ -113,3 +113,22 @@
     </joint>
   </ros2_control>
+  <ros2_control name="ombot_gripper" type="system">
+      <hardware>
+        <plugin>ombot_hardware/OMBotGripperHardware</plugin>
+        <param name="port">/dev/gripper_u2d2</param>
+        <param name="baudrate">1000000</param>
+        <param name="id">12</param>
+        <param name="open_pulse">1754</param>
+        <param name="close_pulse">594</param>
+        <param name="current_limit_mA">300</param>
+        <param name="simulate">false</param>
+      </hardware>
+      <joint name="gripper_joint">
+        <command_interface name="position"/>
+        <command_interface name="effort"/>
+        <state_interface name="position"/>
+        <state_interface name="velocity"/>
+        <state_interface name="effort"/>
+      </joint>
+    </ros2_control>
 </robot>

Commit message: the rviz is mostly updated except the base of the link7 needs to be replaced with the custom designed connector

File: src/ombot_description/urdf/arm/ombot_arm_description.urdf.xacro (robot description, xacro)
@@ -241,4 +241,101 @@
     </inertial>
   </link>
+  <!-- Gripper body (fixed to end_link) -->
+  <link name="gripper_main_link">
+    <visual>
+      <origin xyz="0 0 0" rpy="0 0 0"/>
+      <geometry>
+        <mesh filename="package://ombot_description/meshes/arm/link7.stl" scale="0.001 0.001 0.001"/>
+      </geometry>
+      <material name="grey"/>
+    </visual>
+    <collision>
+      <origin xyz="0 0 0" rpy="0 0 0"/>
+      <geometry>
+        <mesh filename="package://ombot_description/meshes/arm/link7.stl" scale="0.001 0.001 0.001"/>
+      </geometry>
+    </collision>
+    <inertial>
+      <origin xyz="0 0 0" rpy="0 0 0"/>
+      <mass value="0.10"/>
+      <inertia ixx="0.0001" ixy="0" ixz="0" iyy="0.0001" iyz="0" izz="0.0001"/>
+    </inertial>
+  </link>
+  <joint name="gripper_base_joint" type="fixed">
+    <parent link="end_link"/>
+    <child link="gripper_main_link"/>
+    <origin xyz="0 0 0" rpy="${pi/2} 0 0"/>
+  </joint>
+  <!-- Active finger -->
+  <link name="gripper_link">
+    <visual>
+      <origin xyz="0 0 0" rpy="0 0 0"/>
+      <geometry>
+        <mesh filename="package://ombot_description/meshes/arm/gripper_left_palm.stl" scale="0.001 0.001 0.001"/>
+      </geometry>
+      <material name="grey"/>
+    </visual>
+    <collision>
+      <origin xyz="0 0 0" rpy="0 0 0"/>
+      <geometry>
+        <mesh filename="package://ombot_description/meshes/arm/gripper_left_palm.stl" scale="0.001 0.001 0.001"/>
+      </geometry>
+    </collision>
+    <inertial>
+      <origin xyz="0 0 0" rpy="0 0 0"/>
+      <mass value="0.05"/>
+      <inertia ixx="0.00005" ixy="0" ixz="0" iyy="0.00005" iyz="0" izz="0.00005"/>
+    </inertial>
+  </link>
+  <joint name="gripper_joint" type="prismatic">
+    <parent link="gripper_main_link"/>
+    <child link="gripper_link"/>
+    <origin xyz="0.0817 0.021 0.0" rpy="0 0 0"/>
+    <axis xyz="0 1 0"/>
+    <limit lower="-0.010" upper="0.019" effort="10" velocity="1.0"/>
+    <dynamics damping="0.1"/>
+  </joint>
+  <!-- Mirrored finger (display only, mimics gripper_joint) -->
+  <link name="gripper_sub_link">
+    <visual>
+      <origin xyz="0 0 0" rpy="0 0 0"/>
+      <geometry>
+        <mesh filename="package://ombot_description/meshes/arm/gripper_right_palm.stl" scale="0.001 0.001 0.001"/>
+      </geometry>
+      <material name="grey"/>
+    </visual>
+    <collision>
+      <origin xyz="0 0 0" rpy="0 0 0"/>
+      <geometry>
+        <mesh filename="package://ombot_description/meshes/arm/gripper_right_palm.stl" scale="0.001 0.001 0.001"/>
+      </geometry>
+    </collision>
+    <inertial>
+      <origin xyz="0 0 0" rpy="0 0 0"/>
+      <mass value="0.05"/>
+      <inertia ixx="0.00005" ixy="0" ixz="0" iyy="0.00005" iyz="0" izz="0.00005"/>
+    </inertial>
+  </link>
+  <joint name="gripper_sub_joint" type="prismatic">
+    <parent link="gripper_main_link"/>
+    <child link="gripper_sub_link"/>
+    <origin xyz="0.0817 -0.021 0.0" rpy="0 0 0"/>
+    <axis xyz="0 -1 0"/>
+    <limit lower="-0.010" upper="0.019" effort="10" velocity="1.0"/>
+    <dynamics damping="0.1"/>
+    <mimic joint="gripper_joint" multiplier="1" offset="0"/>
+  </joint>
+  <joint name="end_effector_joint" type="fixed">
+    <parent link="gripper_main_link"/>
+    <child link="end_effector_link"/>
+    <origin xyz="0.126 0.0 0.0" rpy="0 0 0"/>
+  </joint>
+  <link name="end_effector_link">
+    <visual>
+      <origin xyz="0 0 0" rpy="0 0 0"/>
+      <geometry><box size="0.01 0.01 0.01"/></geometry>
+      <material name="red"><color rgba="1.0 0.0 0.0 1"/></material>
+    </visual>
+  </link>
 </xacro:macro>
 </robot>

Commit message: Checkpoint from VS Code for cloud agent session

File: src/ombot_description/urdf/arm/ombot_arm_description.urdf.xacro (robot description, xacro)
@@ -186,28 +186,4 @@
     </inertial>
   </link>
-  <!-- Camera body frame mounted to link_6 -->
-  <link name="camera_link">
-    <visual>
-      <origin xyz="0 0 0" rpy="0 0 0"/>
-      <geometry>
-        <box size="0.055 0.135 0.03"/>
-      </geometry>
-      <material name="black"/>
-    </visual>
-  </link>
-  <joint name="camera_mount_joint" type="fixed">
-    <parent link="link_6"/>
-    <!-- Adjust these to your actual bracket offsets on link_6 -->
-    <child link="camera_link"/>
-    <origin xyz="0.08 -0.045 -0.035" rpy="0 0 0"/>
-  </joint>
-  <!-- Standard ROS optical frame: z forward, x right, y down (REP 103) -->
-  <link name="camera_optical_frame"/>
-  <joint name="camera_optical_joint" type="fixed">
-    <parent link="camera_link"/>
-    <child link="camera_optical_frame"/>
-    <!-- This rotation converts a conventional 'camera_link' to an optical frame -->
-    <origin xyz="0 0 0" rpy="-1.57079632679 0 -1.57079632679"/>
-  </joint>
   <!-- Joint 6 -->
   <joint name="joint_6" type="revolute">

File: src/ombot_description/urdf/base/mecanum_base.urdf.xacro (robot description, xacro)
@@ -11,5 +11,5 @@
       <xacro:include filename="/home/frank/frank_ws/src/ombot_description/urdf/base/mech/robot_3d_base.urdf.xacro"/>
       <xacro:include filename="/home/frank/frank_ws/src/ombot_description/urdf/base/mech/mecanum_wheel.urdf.xacro"/>
-      <xacro:include filename="/home/frank/frank_ws/src/ombot_description/urdf/base/sensors/rgbd_camera.urdf.xacro"/>
+      <!-- <xacro:include filename="/home/frank/frank_ws/src/ombot_description/urdf/base/sensors/rgbd_camera.urdf.xacro"/> -->
       <xacro:include filename="/home/frank/frank_ws/src/ombot_description/urdf/base/sensors/lidar.urdf.xacro"/>
       <xacro:include filename="/home/frank/frank_ws/src/ombot_description/urdf/base/sensors/imu.urdf.xacro"/>
@@ -42,9 +42,9 @@
         x_reflect="-1"
         y_reflect="-1"/>
-      <xacro:rgbd_camera
+      <!-- <xacro:rgbd_camera
         prefix="$(arg prefix)"
         camera_name="cam_1"
         xyz_offset="0.105 0 0.03"
-        rpy_offset="0 0 0"/>
+        rpy_offset="0 0 0"/> -->
       <!-- <xacro:lidar_sensor
         prefix="$(arg prefix)"

File: src/ombot_description/urdf/ombot.urdf.xacro (robot description, xacro)
@@ -132,3 +132,13 @@
       </joint>
     </ros2_control>
+  <!-- ZED 2 camera mounted to base_link -->
+  <xacro:include filename="$(find ombot_description)/urdf/zed_macro.urdf.xacro"/>
+  <xacro:zed_camera name="zed2" model="zed2">
+    <origin xyz="0 0 0" rpy="0 0 0"/>
+  </xacro:zed_camera>
+  <joint name="zed2_camera_mount_joint" type="fixed">
+    <parent link="base_link"/>
+    <child link="zed2_camera_link"/>
+    <origin xyz="0.22 0.12 0.13" rpy="0 -0.05 ${-pi/2}"/>
+  </joint>
 </robot>

File: src/ombot_description/urdf/ombot_sim.urdf.xacro (robot description, xacro)
@@ -2,8 +2,8 @@
 <robot name="ombot" xmlns:xacro="http://www.ros.org/wiki/xacro">
   <!-- Base geometry -->
-  <xacro:include filename="/home/frank/frank_ws/src/ombot_description/urdf/base/mecanum_base.urdf.xacro"/>
+  <xacro:include filename="$(find ombot_description)/urdf/base/mecanum_base.urdf.xacro"/>
   <xacro:mecanum_base prefix="" sep_x="0.40" sep_y="0.70" wheel_radius="0.05"/>
   <!-- Arm geometry -->
-  <xacro:include filename="/home/frank/frank_ws/src/ombot_description/urdf/arm/ombot_arm_module.urdf.xacro"/>
+  <xacro:include filename="$(find ombot_description)/urdf/arm/ombot_arm_module.urdf.xacro"/>
   <xacro:ombot_arm_module parent="base_link" mount_xyz="0.145 0.0 0.1" mount_rpy="0 0 0" prefix=""/>
   <!-- BASE: mock hardware -->
@@ -94,3 +94,13 @@
     </joint>
   </ros2_control>
+  <!-- ZED 2 camera mounted to base_link -->
+  <xacro:include filename="$(find ombot_description)/urdf/zed_macro.urdf.xacro"/>
+  <xacro:zed_camera name="zed2" model="zed2">
+    <origin xyz="0 0 0" rpy="0 0 0"/>
+  </xacro:zed_camera>
+  <joint name="zed2_camera_mount_joint" type="fixed">
+    <parent link="base_link"/>
+    <child link="zed2_camera_link"/>
+    <origin xyz="0.22 0.12 0.13" rpy="0 -0.05 ${-pi/2}"/>
+  </joint>
 </robot>
